File: Hardware/PCBs/1_keyboard/OpenRPNCalc_keyboard.kicad_sch (KiCad schematic)
At the start: 46 parts, among them J1 AMPHENOL F32R-1A7H1-11020, SW1 "0", SW10 "-", SW11 "4", SW12 "5", SW13 "6", SW14 "*", SW15 "/", SW16 "7", SW17 "8", SW18 "9", SW19 "EXP", SW2 "/-/", SW20 "C", SW21 "sqrt", SW22 "1/x", SW23 "erf", SW24 "R->P", SW25 "Gamma(x)", SW26 "Cxy", SW27 "y^x", SW28 "ln", SW29 "lg", SW3 ".", SW30 "sin", SW31 "cos", SW32 "tan", SW33 "Drop", SW34 "X<>Y", SW35 "DR", SW36 "M+", SW37 "MR", SW38 "MS", SW39 "F", SW4 "+-", SW40 "G", SW41 "Mode", SW42 "Uncr", SW43 Prec, SW44 "On", SW5 "Enter", SW6 "1", SW7 "2", SW8 "3", SW9 "+"

Commit message: Update to rev 3.1
Parts:
- BT1: value 3V -> BLP2016SM-GTR
- SW1: value "0" -> EVPBT1C4A000
- SW10: value "-" -> EVPBT1C4A000
- SW11: value "4" -> EVPBT1C4A000
- SW12: value "5" -> EVPBT1C4A000
- SW13: value "6" -> EVPBT1C4A000
- SW14: value "*" -> EVPBT1C4A000
- SW15: value "/" -> EVPBT1C4A000
- SW16: value "7" -> EVPBT1C4A000
- SW17: value "8" -> EVPBT1C4A000
- SW18: value "9" -> EVPBT1C4A000
- SW19: value "EXP" -> EVPBT1C4A000
- SW2: value "/-/" -> EVPBT1C4A000
- SW20: value "C" -> EVPBT1C4A000
- SW21: value "sqrt" -> EVPBT1C4A000
- SW22: value "1/x" -> EVPBT1C4A000
- SW23: value "erf" -> EVPBT1C4A000
- SW24: value "R->P" -> EVPBT1C4A000
- SW25: value "Gamma(x)" -> EVPBT1C4A000
- SW26: value "Cxy" -> EVPBT1C4A000
- SW27: value "y^x" -> EVPBT1C4A000
- SW28: value "ln" -> EVPBT1C4A000
- SW29: value "lg" -> EVPBT1C4A000
- SW3: value "." -> EVPBT1C4A000
- SW30: value "sin" -> EVPBT1C4A000
- SW31: value "cos" -> EVPBT1C4A000
- SW32: value "tan" -> EVPBT1C4A000
- SW33: value "Drop" -> EVPBT1C4A000
- SW34: value "X<>Y" -> EVPBT1C4A000
- SW35: value "DR" -> EVPBT1C4A000
- SW36: value "M+" -> EVPBT1C4A000
- SW37: value "MR" -> EVPBT1C4A000
- SW38: value "MS" -> EVPBT1C4A000
- SW39: value "F" -> EVPBT1C4A000
- SW4: value "+-" -> EVPBT1C4A000
- SW40: value "G" -> EVPBT1C4A000
- SW41: value "Mode" -> EVPBT1C4A000
- SW42: value "Uncr" -> EVPBT1C4A000
- SW43: value Prec -> EVPBT1C4A000
- SW44: value "On" -> EVPBT1C4A000
- SW5: value "Enter" -> EVPBT1C4A000
- SW6: value "1" -> EVPBT1C4A000
- SW7: value "2" -> EVPBT1C4A000
- SW8: value "3" -> EVPBT1C4A000
- SW9: value "+" -> EVPBT1C4A000
Connections:
- no-connect marks 1 -> 2
