File: Hardware/PCBs/4_MCU/OpenRPNCalc_MCU.kicad_pcb (KiCad board)
At the start: 2 copper layers, 73 x 134.4 mm, 51 parts, among them J1 HARWIN M22-5330505, J2 Molex 5051101092, J3 F32R-1A7H1-11020, SW45 EVQP0N02B, SW46 Nidec CUS-12TB, U1 TPS61222DCK, U2 STM32L476RETx, Y1 32768 Hz

Commit message: Update to rev 3.1
Parts:
- D1: footprint Diode_SMD:D_SOD-323_HandSoldering -> Diode_SMD:D_0603_1608Metric_Pad1.05x0.95mm_HandSolder
- SW45: value EVQP0N02B -> EVQQ2P03W
Routing:
- net Net-(D1-K): track 25.5 -> 24.8 mm
Other:
- board text removed: "Display area"
Changed lines of the file:
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@@
     )
   )
-  (footprint "Diode_SMD:D_SOD-323_HandSoldering" placed (layer "B.Cu")
+  (footprint "Diode_SMD:D_0603_1608Metric_Pad1.05x0.95mm_HandSolder" (layer "B.Cu")
     (at 72.7 48.3 -90)
-    (descr "SOD-323")
-    (tags "SOD-323")
+    (descr "Diode SMD 0603 (1608 Metric), square (rectangular) end terminal, IPC_7351 nominal, (Body size source: http://www.tortai-tech.com/upload/download/2011102023233369053.pdf), generated with kicad-footprint-generator")
+    (tags "diode handsolder")
     (property "Sheetfile" "OpenRPNCalc_MCU.kicad_sch")
     (property "Sheetname" "")
@@
     (property "ki_keywords" "diode Schottky")
     (attr smd)
-    (fp_text reference "D1" (at 0 1.85 -270) (layer "B.SilkS")
+    (fp_text reference "D1" (at 0 1.43 90) (layer "B.SilkS")
         (effects (font (size 1 1) (thickness 0.15)) (justify mirror))
     )
-    (fp_text value "NSR0340HT1G" (at 0.4 3.4 -270) (layer "B.Fab")
+    (fp_text value "NSR0340HT1G" (at 0 -1.43 90) (layer "B.Fab")
         (effects (font (size 1 1) (thickness 0.15)) (justify mirror))
     )
-    (fp_text user "${REFERENCE}" (at 0 1.85 -270) (layer "B.Fab")
-        (effects (font (size 1 1) (thickness 0.15)) (justify mirror))
+    (fp_text user "${REFERENCE}" (at 0 0 90) (layer "B.Fab")
+        (effects (font (size 0.4 0.4) (thickness 0.06)) (justify mirror))
     )
-    (fp_line (start -2.01 -0.85) (end 1.25 -0.85)
+    (fp_line (start -1.66 -0.735) (end 0.8 -0.735)
       (stroke (width 0.12) (type solid)) (layer "B.SilkS"))
-    (fp_line (start -2.01 0.85) (end -2.01 -0.85)
+    (fp_line (start -1.66 0.735) (end -1.66 -0.735)
       (stroke (width 0.12) (type solid)) (layer "B.SilkS"))
-    (fp_line (start -2.01 0.85) (end 1.25 0.85)
+    (fp_line (start 0.8 0.735) (end -1.66 0.735)
       (stroke (width 0.12) (type solid)) (layer "B.SilkS"))
-    (fp_line (start -2 -0.95) (end 2 -0.95)
+    (fp_line (start -1.65 -0.73) (end -1.65 0.73)
       (stroke (width 0.05) (type solid)) (layer "B.CrtYd"))
-    (fp_line (start -2 0.95) (end -2 -0.95)
+    (fp_line (start -1.65 0.73) (end 1.65 0.73)
       (stroke (width 0.05) (type solid)) (layer "B.CrtYd"))
-    (fp_line (start -2 0.95) (end 2 0.95)
+    (fp_line (start 1.65 -0.73) (end -1.65 -0.73)
       (stroke (width 0.05) (type solid)) (layer "B.CrtYd"))
-    (fp_line (start 2 0.95) (end 2 -0.95)
+    (fp_line (start 1.65 0.73) (end 1.65 -0.73)
       (stroke (width 0.05) (type solid)) (layer "B.CrtYd"))
-    (fp_line (start -0.9 -0.7) (end -0.9 0.7)
+    (fp_line (start -0.8 -0.4) (end 0.8 -0.4)
       (stroke (width 0.1) (type solid)) (layer "B.Fab"))
-    (fp_line (start -0.9 0.7) (end 0.9 0.7)
+    (fp_line (start -0.8 0.1) (end -0.8 -0.4)
       (stroke (width 0.1) (type solid)) (layer "B.Fab"))
-    (fp_line (start -0.3 0) (end -0.5 0)
+    (fp_line (start -0.5 0.4) (end -0.8 0.1)
       (stroke (width 0.1) (type solid)) (layer "B.Fab"))
-    (fp_line (start -0.3 0) (end 0.2 0.35)
+    (fp_line (start 0.8 -0.4) (end 0.8 0.4)
       (stroke (width 0.1) (type solid)) (layer "B.Fab"))
-    (fp_line (start -0.3 0.35) (end -0.3 -0.35)
+    (fp_line (start 0.8 0.4) (end -0.5 0.4)
       (stroke (width 0.1) (type solid)) (layer "B.Fab"))
-    (fp_line (start 0.2 -0.35) (end -0.3 0)
-      (stroke (width 0.1) (type solid)) (layer "B.Fab"))
-    (fp_line (start 0.2 0) (end 0.45 0)
-      (stroke (width 0.1) (type solid)) (layer "B.Fab"))
-    (fp_line (start 0.2 0.35) (end 0.2 -0.35)
-      (stroke (width 0.1) (type solid)) (layer "B.Fab"))
-    (fp_line (start 0.9 -0.7) (end -0.9 -0.7)
-      (stroke (width 0.1) (type solid)) (layer "B.Fab"))
-    (fp_line (start 0.9 0.7) (end 0.9 -0.7)
-      (stroke (width 0.1) (type solid)) (layer "B.Fab"))
-    (pad "1" smd roundrect (at -1.25 0 270) (size 1 1) (layers "B.Cu" "B.Paste" "B.Mask") (roundrect_rratio 0.25)
+    (pad "1" smd roundrect (at -0.875 0 270) (size 1.05 0.95) (layers "B.Cu" "B.Paste" "B.Mask") (roundrect_rratio 0.25)
       (net 32 "Net-(D1-K)") (pinfunction "K") (pintype "passive"))
-    (pad "2" smd roundrect (at 1.25 0 270) (size 1 1) (layers "B.Cu" "B.Paste" "B.Mask") (roundrect_rratio 0.25)
+    (pad "2" smd roundrect (at 0.875 0 270) (size 1.05 0.95) (layers "B.Cu" "B.Paste" "B.Mask") (roundrect_rratio 0.25)
       (net 35 "Net-(D1-A)") (pinfunction "A") (pintype "passive"))
-    (model "${KICAD6_3DMODEL_DIR}/Diode_SMD.3dshapes/D_SOD-323.wrl"
+    (model "${KICAD6_3DMODEL_DIR}/Diode_SMD.3dshapes/D_0603_1608Metric.wrl"
       (offset (xyz 0 0 0))
       (scale (xyz 1 1 1))
@@
         (effects (font (size 1 1) (thickness 0.15)) (justify mirror))
     )
-    (fp_text value "EVQP0N02B" (at 0 -4.25) (layer "B.Fab")
+    (fp_text value "EVQQ2P03W" (at 0 -4.25) (layer "B.Fab")
         (effects (font (size 1 1) (thickness 0.15)) (justify mirror))
     )
@@
     )
   )
-  (gr_line (start 129.7 74) (end 88.3 74)
-    (stroke (width 0.12) (type default)) (layer "F.SilkS"))
-  (gr_line (start 74.9 74) (end 69.7 74)
-    (stroke (width 0.12) (type default)) (layer "F.SilkS"))
   (gr_rect (start 68.195712 36) (end 131.195712 79)
     (stroke (width 0.12) (type default)) (fill none) (layer "F.SilkS"))
-  (gr_line (start 129.7 38) (end 129.7 74)
-    (stroke (width 0.12) (type default)) (layer "F.SilkS"))
-  (gr_line (start 69.7 38) (end 129.7 38)
-    (stroke (width 0.12) (type default)) (layer "F.SilkS"))
-  (gr_line (start 69.7 74) (end 69.7 38)
-    (stroke (width 0.12) (type default)) (layer "F.SilkS"))
   (gr_circle (center 130.7 104.1) (end 130.7 103.8)
     (stroke (width 0.05) (type default)) (fill none) (layer "Edge.Cuts"))
@@
     (effects (font (size 1 1) (thickness 0.15)) (justify left bottom))
   )
-  (gr_text "Display area" (at 69.8 39.6) (layer "F.SilkS")
-    (effects (font (size 1 1) (thickness 0.15)) (justify left bottom))
-  )
   (gr_text "Rev 3.1" (at 123 42.5) (layer "F.SilkS")
     (effects (font (size 1 1) (thickness 0.15)) (justify left bottom))
@@
   (segment (start 88.5375 81.3375) (end 88.7 81.5) (width 0.25) (layer "B.Cu") (net 31))
   (segment (start 83.5872 36.0216) (end 72.3784 36.0216) (width 0.5) (layer "B.Cu") (net 32))
-  (segment (start 70.8 37.6) (end 70.8 45.15) (width 0.5) (layer "B.Cu") (net 32))
-  (segment (start 70.8 45.15) (end 72.7 47.05) (width 0.5) (layer "B.Cu") (net 32))
+  (segment (start 72.7 46.5) (end 72.7 47.05) (width 0.5) (layer "B.Cu") (net 32))
   (segment (start 83.5872 34.9454) (end 83.5872 36.0216) (width 0.5) (layer "B.Cu") (net 32))
+  (segment (start 70.8 37.6) (end 70.8 44.6) (width 0.5) (layer "B.Cu") (net 32))
+  (segment (start 70.8 44.6) (end 72.7 46.5) (width 0.5) (layer "B.Cu") (net 32))
   (segment (start 72.3784 36.0216) (end 70.8 37.6) (width 0.5) (layer "B.Cu") (net 32))
-  (segment (start 73.1978 46.5522) (end 72.7 47.05) (width 0.25) (layer "B.Cu") (net 32))
   (segment (start 94.375 40.65) (end 94.3 40.725) (width 0.25) (layer "B.Cu") (net 33))
   (segment (start 96.4 40.65) (end 94.375 40.65) (width 0.5) (layer "B.Cu") (net 33))
@@
   (segment (start 115.85 75.65) (end 115.85 77.225) (width 0.25) (layer "B.Cu") (net 34))
   (segment (start 115.85 77.225) (end 117.6 78.975) (width 0.25) (layer "B.Cu") (net 34))
-  (segment (start 74 42.1694) (end 74 48.25) (width 0.5) (layer "B.Cu") (net 35))
   (segment (start 72.1 40.2694) (end 74 42.1694) (width 0.5) (layer "B.Cu") (net 35))
-  (segment (start 74 48.25) (end 72.7 49.55) (width 0.5) (layer "B.Cu") (net 35))
+  (segment (start 72.925 49.175) (end 72.7 49.175) (width 0.5) (layer "B.Cu") (net 35))
+  (segment (start 74 48.1) (end 72.925 49.175) (width 0.5) (layer "B.Cu") (net 35))
+  (segment (start 74 42.1694) (end 74 48.1) (width 0.5) (layer "B.Cu") (net 35))
   (segment (start 72.1 38.9275) (end 72.1 40.2694) (width 0.5) (layer "B.Cu") (net 35))
   (segment (start 120.077997 61.622003) (end 120.9749 62.518906) (width 0.25) (layer "F.Cu") (net 62))
