File: Hardware/PCBs/4_MCU/OpenRPNCalc_MCU.kicad_sch (KiCad schematic)
At the start: 51 parts, among them J1 HARWIN M22-5330505, J2 Molex 5051101092, J3 F32R-1A7H1-11020, SW45 EVQP0N02B, SW46 Nidec CUS-12TB, U1 TPS61222DCK, U2 STM32L476RETx, Y1 32768 Hz

Commit message: Update to rev 3.1
Parts:
- SW45: value EVQP0N02B -> EVQQ2P03W
Changed lines of the file:
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@@
   (title_block
     (title "OpenRPNCalc")
-    (date "2025-02-09")
-    (rev "3.0")
+    (date "2025-03-08")
+    (rev "3.1")
   )
   (junction (at 107.95 146.05) (diameter 0) (color 0 0 0 0)
@@
       (effects (font (size 1.27 1.27)) (justify left))
     )
-    (property "Value" "EVQP0N02B" (at 25.4508 37.973 90)
+    (property "Value" "EVQQ2P03W" (at 25.4508 37.973 90)
       (effects (font (size 1.27 1.27)) (justify left))
     )
