File: Hardware/PCBs/Main/main.kicad_sch (KiCad schematic)
At the start: 137 parts, among them J2 HARWIN M20, J3 USB4110GFA, J4 F3311A7H121010E200, SW1 EVQQ2P03W, SW10 EVPBT1C4A000, SW11 EVPBT1C4A000, SW12 EVPBT1C4A000, SW13 EVPBT1C4A000, SW14 EVPBT1C4A000, SW15 EVPBT1C4A000, SW16 EVPBT1C4A000, SW17 EVPBT1C4A000, SW18 EVPBT1C4A000, SW19 EVPBT1C4A000, SW2 Nidec CUS-12TB, SW20 EVPBT1C4A000, SW21 EVPBT1C4A000, SW22 EVPBT1C4A000, SW23 EVPBT1C4A000, SW24 EVPBT1C4A000, SW25 EVPBT1C4A000, SW26 EVPBT1C4A000, SW27 EVPBT1C4A000, SW28 EVPBT1C4A000, SW29 EVPBT1C4A000, SW3 EVPBT1C4A000, SW30 EVPBT1C4A000, SW31 EVPBT1C4A000, SW32 EVPBT1C4A000, SW33 EVPBT1C4A000, SW34 EVPBT1C4A000, SW35 EVPBT1C4A000, SW36 EVPBT1C4A000, SW37 EVPBT1C4A000, SW38 EVPBT1C4A000, SW39 EVPBT1C4A000, SW4 EVPBT1C4A000, SW40 EVPBT1C4A000, SW41 EVPBT1C4A000, SW42 EVPBT1C4A000, SW43 EVPBT1C4A000, SW44 EVPBT1C4A000, SW45 EVPBT1C4A000, SW46 EVPBT1C4A000, SW47 EVPBT1C4A000, SW48 EVPBT1C4A000, SW49 EVPBT1C4A000, SW5 EVPBT1C4A000, SW50 EVPBT1C4A000, SW51 EVPBT1C4A000, SW6 EVPBT1C4A000, SW7 EVPBT1C4A000, SW8 EVPBT1C4A000, SW9 EVPBT1C4A000, U1 STM32U385RGT6Q, U2 TPS61299, U3 MX25R6435FM2IL0, U4 TLV73333PDBVR, U5 LM66100QDCKRQ1, U6 LM66100QDCKRQ1, U7 NBM5100A, Y1 32768 Hz

Commit message: Update rev 4 schematics
Parts:
- added JP1: Bootloader, Resistor_SMD:R_0603_1608Metric_Pad0.98x0.95mm_HandSolder, symbol Jumper:Jumper_2_Open
- added R29, R30: 33, Resistor_SMD:R_0603_1608Metric_Pad0.98x0.95mm_HandSolder, symbol Device:R
- added R31: 0, Resistor_SMD:R_0603_1608Metric_Pad0.98x0.95mm_HandSolder, symbol Device:R
- R25: value 100 -> 0
Connections:
- net SWCLK: now also R29.2
- net SWDIO: now also R30.2
- net VDD: now also JP1.1 (A), R31.2
- net at R2.1, U1.60 (PH3-BOOT0): now also JP1.2 (B)
- net at C24.1, D3.2 (A), R22.1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: now also R31.1
- net at J3.A8 (SBU1): now also R29.1
- net at J3.B8 (SUB2): now also R30.1
- no-connect marks 5 -> 8
Other:
- moved on the sheet: BT1, C1, C10, C11, C12, C13, C14, C15, C16, C17, C18, C19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

Commit message: Update component names in schematic, add PDBs
Parts:
- C24, C25: value 2 uF -> 2.2 uF
- J2: value HARWIN M20 -> HARWIN M20-8890545R
- J3: value USB4110GFA -> USB4110-GF-A
- SW1: value EVQQ2P03W -> TL1014BF160QG
- SW2: value Nidec CUS-12TB -> CUS-12TB
- TP1, TP10, TP11, TP12, TP13, TP2, TP3, TP4, TP5, TP6, TP7, TP8, TP9: footprint TestPoint:TestPoint_Pad_D2.0mm -> footprints:TestPoint_Pad_D2.0mm
- U2: value TPS61299 -> TPS61299DRLR
Connections:
- no-connect marks 8 -> 9
Other:
- moved on the sheet: SW10, SW11, SW12, SW13, SW14, SW15, SW16, SW17, SW18, SW19, SW20, SW21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
