File: Hardware/PCBs/Spacer2/Spacer2_assembly.kicad_pcb (KiCad board)
At the start: 2 copper layers, 73 x 139 mm, 0 parts

Commit message: Bugfix 4.0; added HP48 layout
Other:
- outline, holes or cut-outs redrawn
Changed lines of the file:
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@@
-		(layer "Edge.Cuts")
-	)
-	(gr_circle
-		(center 43.185793 79.692893)
-		(end 44.285793 79.692893)
-		(stroke
-			(width 0.05)
-			(type default)
-		)
-		(fill no)
 		(layer "Edge.Cuts")
 	)
@@
 		(layer "Edge.Cuts")
 	)
-	(gr_line
-		(start 39.985793 82.892893)
-		(end 59.285793 82.892893)
-		(stroke
-			(width 0.05)
-			(type default)
-		)
-		(layer "Edge.Cuts")
-	)
 	(gr_circle
 		(center 42.7 109.5)
@@
 		(layer "Edge.Cuts")
 	)
-	(gr_line
-		(start 39.985793 58.692893)
-		(end 59.285793 58.692893)
-		(stroke
-			(width 0.05)
-			(type default)
-		)
-		(layer "Edge.Cuts")
-	)
 	(gr_arc
 		(start 59.2 48)
@@
 	)
 	(gr_line
-		(start 60.285793 61.992893)
-		(end 60.285793 59.692893)
-		(stroke
-			(width 0.05)
-			(type default)
-		)
-		(layer "Edge.Cuts")
-	)
-	(gr_line
 		(start 80.1 45.8)
 		(end 80.1 43)
@@
 		(layer "Edge.Cuts")
 	)
-	(gr_arc
-		(start 60.285793 81.892893)
-		(mid 59.9929 82.6)
-		(end 59.285793 82.892893)
-		(stroke
-			(width 0.05)
-			(type default)
-		)
-		(layer "Edge.Cuts")
-	)
 	(gr_line
 		(start 84.9 56.9)
@@
 	)
 	(gr_line
-		(start 39.985793 58.692893)
-		(end 39.985793 82.892893)
-		(stroke
-			(width 0.05)
-			(type default)
-		)
-		(layer "Edge.Cuts")
-	)
-	(gr_line
 		(start 108 89.9)
 		(end 107.999999 92.399999)
@@
 	)
 	(gr_arc
-		(start 59.285793 58.692893)
-		(mid 59.9929 58.985786)
-		(end 60.285793 59.692893)
-		(stroke
-			(width 0.05)
-			(type default)
-		)
-		(layer "Edge.Cuts")
-	)
-	(gr_arc
 		(start 45 89.9)
 		(mid 45.292893 89.192893)
@@
 	)
 	(gr_line
-		(start 60.285793 79.592892)
-		(end 60.285793 81.892893)
-		(stroke
-			(width 0.05)
-			(type default)
-		)
-		(layer "Edge.Cuts")
-	)
-	(gr_line
 		(start 102.3 69.1)
 		(end 98.3 69.1)
@@
 		(layer "Edge.Cuts")
 	)
-	(gr_arc
-		(start 60.285793 79.592893)
-		(mid 44.713013 70.792893)
-		(end 60.285793 61.992892)
-		(stroke
-			(width 0.05)
-			(type default)
-		)
-		(layer "Edge.Cuts")
-	)
 	(gr_line
 		(start 94.5 48.6)
@@
 		(layer "Edge.Cuts")
 	)
-	(gr_circle
-		(center 43.185793 61.892893)
-		(end 44.285793 61.892893)
-		(stroke
-			(width 0.05)
-			(type default)
-		)
-		(fill no)
-		(layer "Edge.Cuts")
-	)
