File: Hardware/PCBs/Spacer2/Spacer2_production.kicad_pcb (KiCad board)
At the start: 2 copper layers, 73 x 139 mm, 0 parts

Commit message: Bugfix 4.0; added HP48 layout
Other:
- outline, holes or cut-outs redrawn
Changed lines of the file:
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@@
-		(layer "Edge.Cuts")
-	)
-	(gr_arc
-		(start 48.59902 83.6)
-		(mid 48.500482 83.595136)
-		(end 48.402904 83.580581)
-		(stroke
-			(width 0.05)
-			(type default)
-		)
 		(layer "Edge.Cuts")
 	)
@@
 		(layer "Edge.Cuts")
 	)
-	(gr_line
-		(start 58.8 57.996446)
-		(end 60 58)
+	(gr_arc
+		(start 48.440555 57.655033)
+		(mid 48.60184 57.613854)
+		(end 48.767721 57.6)
+		(stroke
+			(width 0.12)
+			(type default)
+		)
+		(layer "Edge.Cuts")
+	)
+	(gr_line
+		(start 58.8 57.598223)
+		(end 60 57.601777)
 		(stroke
 			(width 0.12)
@@
 	)
 	(gr_line
-		(start 58.803553 83.603554)
-		(end 59.9929 83.599993)
+		(start 58.80049 84)
+		(end 59.9929 84)
 		(stroke
 			(width 0.12)
@@
 	)
 	(gr_arc
-		(start 82 135.9)
-		(mid 82.292893 135.192893)
-		(end 83 134.9)
+		(start 82 136.9)
+		(mid 82.292893 136.192893)
+		(end 83 135.9)
 		(stroke
 			(width 0.05)
@@
 	)
 	(gr_arc
-		(start 48.402904 58.019419)
-		(mid 48.500482 58.004867)
-		(end 48.59902 58)
-		(stroke
-			(width 0.12)
-			(type default)
-		)
-		(layer "Edge.Cuts")
-	)
-	(gr_arc
 		(start 80.500008 123.900008)
 		(mid 80.792899 123.192899)
@@
 	)
 	(gr_line
-		(start 58.8 83.6)
-		(end 48.59902 83.6)
+		(start 58.80049 84)
+		(end 48.767721 84)
 		(stroke
 			(width 0.05)
@@
 	)
 	(gr_line
-		(start 89 142.4)
+		(start 88.6 142.4)
 		(end 105 142.4)
 		(stroke
@@
 	)
 	(gr_arc
-		(start 59.999993 58.000007)
-		(mid 60.707102 58.292898)
-		(end 60.999993 59.000007)
-		(stroke
-			(width 0.12)
-			(type default)
-		)
-		(layer "Edge.Cuts")
-	)
-	(gr_arc
-		(start 88 136.4)
-		(mid 88.707107 136.692893)
-		(end 89 137.4)
+		(start 59.999993 57.601784)
+		(mid 60.707102 57.894675)
+		(end 60.999993 58.601784)
+		(stroke
+			(width 0.12)
+			(type default)
+		)
+		(layer "Edge.Cuts")
+	)
+	(gr_arc
+		(start 87.6 137.4)
+		(mid 88.307107 137.692893)
+		(end 88.6 138.4)
 		(stroke
 			(width 0.05)
@@
 	)
 	(gr_circle
-		(center 84.4 155.8)
-		(end 86 155.8)
+		(center 84.4 154.5)
+		(end 86 154.5)
 		(stroke
 			(width 0.05)
@@
 	)
 	(gr_line
-		(start 80 137.4)
-		(end 80 142.4)
-		(stroke
-			(width 0.05)
-			(type default)
-		)
-		(layer "Edge.Cuts")
-	)
-	(gr_line
-		(start 61 78.899998)
-		(end 60.992892 82.599993)
+		(start 80.4 138.4)
+		(end 80.4 142.4)
+		(stroke
+			(width 0.05)
+			(type default)
+		)
+		(layer "Edge.Cuts")
+	)
+	(gr_line
+		(start 61 78.9)
+		(end 60.992892 83)
 		(stroke
 			(width 0.12)
@@
 	)
 	(gr_line
-		(start 60.999575 59.000007)
-		(end 61.007181 62.705325)
+		(start 60.999575 58.601784)
+		(end 61.007181 62.705324)
 		(stroke
 			(width 0.12)
@@
 	)
 	(gr_line
-		(start 87 136.4)
-		(end 88 136.4)
+		(start 87 137.4)
+		(end 87.6 137.4)
 		(stroke
 			(width 0.05)
@@
 	(gr_line
 		(start 73.7 142.4)
-		(end 80 142.4)
+		(end 80.4 142.4)
 		(stroke
 			(width 0.05)
@@
 	)
 	(gr_arc
-		(start 80 137.4)
-		(mid 80.292893 136.692893)
-		(end 81 136.4)
+		(start 80.4 138.4)
+		(mid 80.692893 137.692893)
+		(end 81.4 137.4)
 		(stroke
 			(width 0.05)
@@
 	(gr_line
 		(start 46 83.1)
-		(end 48.402904 83.580581)
+		(end 48.440555 83.944967)
 		(stroke
 			(width 0.12)
@@
 	)
 	(gr_line
-		(start 83 134.9)
-		(end 86 134.9)
+		(start 83 135.9)
+		(end 86 135.9)
 		(stroke
 			(width 0.05)
@@
 	)
 	(gr_circle
-		(center 68.5 155.8)
-		(end 70.1 155.8)
+		(center 68.5 154.9)
+		(end 70.1 154.9)
 		(stroke
 			(width 0.05)
@@
 	(gr_line
 		(start 46 58.5)
-		(end 48.402904 58.019419)
+		(end 48.440555 57.655033)
 		(stroke
 			(width 0.12)
@@
 	)
 	(gr_line
-		(start 81 136.4)
-		(end 82 136.4)
+		(start 81.4 137.4)
+		(end 82 137.4)
 		(stroke
 			(width 0.05)
@@
 		(layer "Edge.Cuts")
 	)
+	(gr_arc
+		(start 48.767721 84)
+		(mid 48.60184 83.986146)
+		(end 48.440555 83.944967)
+		(stroke
+			(width 0.05)
+			(type default)
+		)
+		(layer "Edge.Cuts")
+	)
 	(gr_line
 		(start 73.9 46.8)
@@
 	)
 	(gr_line
-		(start 82 135.9)
-		(end 82 136.4)
+		(start 82 136.9)
+		(end 82 137.4)
 		(stroke
 			(width 0.05)
@@
 	)
 	(gr_arc
-		(start 86 134.9)
-		(mid 86.707107 135.192893)
-		(end 87 135.9)
+		(start 86 135.9)
+		(mid 86.707107 136.192893)
+		(end 87 136.9)
 		(stroke
 			(width 0.05)
@@
 	)
 	(gr_line
-		(start 87 135.9)
-		(end 87 136.4)
+		(start 87 136.9)
+		(end 87 137.4)
 		(stroke
 			(width 0.05)
@@
 	)
 	(gr_line
-		(start 58.8 58)
-		(end 48.59902 58)
+		(start 58.80049 57.6)
+		(end 48.767721 57.6)
 		(stroke
 			(width 0.05)
@@
 	)
 	(gr_line
-		(start 89 137.4)
-		(end 89 142.4)
-		(stroke
-			(width 0.05)
-			(type default)
-		)
-		(layer "Edge.Cuts")
-	)
-	(gr_arc
-		(start 60.992893 82.599993)
-		(mid 60.700002 83.307102)
-		(end 59.992893 83.599993)
-		(stroke
-			(width 0.12)
+		(start 88.6 138.4)
+		(end 88.6 142.4)
+		(stroke
+			(width 0.05)
+			(type default)
+		)
+		(layer "Edge.Cuts")
+	)
+	(gr_arc
+		(start 60.992893 83)
+		(mid 60.700002 83.707109)
+		(end 59.992893 84)
+		(stroke
+			(width 0.12)
